Commit message: final version GEAM with vito-robot

File: model/box.urdf.xacro (robot description, xacro)
@@ -1,22 +1,26 @@
 <?xml version="1.0"?>
 <robot xmlns:xacro="http://www.ros.org/wiki/xacro" name="box">
+	<xacro:macro name="box_inertia_def" params="h w d mass">
+	<inertia ixx="${mass * (w*w+d*d)/ 12}"
+			 iyy="${mass * (h*h+d*d)/ 12}"
+			 izz="${mass * (h*h+w*w) / 12}"
+			 ixy="0" iyz="0" ixz="0"/>
+	</xacro:macro>
 	<link name="box">
 		<inertial>
-			<mass value="10.0"/>
-			<!-- cylindrical shell : Izz=m*r^2; Ixx=Iyy=1/12*m*(6*r^2+h^2) -->
-			<!-- solid cylinder : Izz=(m*r^2)/2; Ixx=Iyy=1/12*m*(3*r^2+h^2) -->
-			<!-- <inertia  ixx="0.002385" ixy="0.00"  ixz="0.00" iyy="0.002385" iyz="0.00" izz="0.00027" />-->
-			<inertia  ixx="20" ixy="0.00"  ixz="0.00" iyy="20" iyz="0.00" izz="20" />
+				<mass value="5.0"/>
+				<origin xyz="0 0 0.005"/>
+				<xacro:box_inertia_def h="0.01" w="0.12" d="0.05" mass="5.0" />
 		</inertial>
 		<visual>
-			<origin xyz="0 0 0" rpy="0 0 0"/>
-			<geometry>
-				<box size="0.10  0.06  0.2"/>
+			<origin xyz="0.0 0.0 0.025" rpy="0 0 0"/>
+			 <geometry>
+		      <box size="0.01  0.12  0.05"/>
 			</geometry>
 		</visual>
 		<collision>
-			<origin xyz="0 0 0" rpy="0 0 0"/>
+			<origin xyz="0.0 0.0 0.025" rpy="0 0 0"/>
 			<geometry>
-				<box size="0.10 0.06 0.2"/>
+				 <box size="0.01  0.12  0.05"/> -->
 			</geometry>
 		</collision>
@@ -25,9 +29,13 @@
       	<material>Gazebo/Blue</material>
            <selfCollide>true</selfCollide>
+           <maxContacts>100</maxContacts>
 		  <gravity>true</gravity>
-		 <!--  <mu1>1.0</mu1>
-		  <mu2>1.0</mu2>
-		  <kp>10000000.0</kp>
-	       <kd>1.0</kd> -->
+	    <mu1>0.5</mu1>
+	     <mu2>0.5</mu2>
+	        <fdir1>0 0 0</fdir1>
+         <maxVel>0.0</maxVel>
+		<kp>1000000000.0</kp>
+	  <kd>10000.0</kd>
+	  <minDepth>0.00</minDepth>
 	  </gazebo>
 </robot>

File: model/cylinder.urdf.xacro (robot description, xacro)
@@ -3,41 +3,45 @@
 	<xacro:macro name="cylinder_inertia_def" params="radius length mass">
 	<inertia ixx="${mass * (3 * radius * radius + length * length) / 12}"
-			 iyy="${mass * radius* radius / 2}"
-			 izz="${mass * (3 * radius * radius + length * length) / 12}"
+			 iyy="${mass * (3 * radius * radius + length * length) / 12}"
+			 izz="${mass * radius* radius / 2}"
 			 ixy="0" iyz="0" ixz="0"/>
 	</xacro:macro>
-	<link name="cylinder">
+	<link name="object_link" type="fixed">
+	    <material>Gazebo/Blue</material>
 		<inertial>
-			<!-- cylindrical shell : Izz=m*r^2; Ixx=Iyy=1/12*m*(6*r^2+h^2) -->
-			<!-- solid cylinder : Izz=(m*r^2)/2; Ixx=Iyy=1/12*m*(3*r^2+h^2) -->
-			<!-- <inertia  ixx="0.002385" ixy="0.00"  ixz="0.00" iyy="0.002385" iyz="0.00" izz="0.00027" /> -->
-				<mass value="1.0"/>
-				<origin xyz="0 0 0.006"/>
-				<xacro:cylinder_inertia_def radius="0.035" length="0.012" mass="1.0" />
+				<mass value="4.0"/>
+				<!--<origin xyz="0 0 0.005"/>
+				<xacro:cylinder_inertia_def radius="0.035" length="0.015" mass="5.0" />-->
+				<origin xyz="0 0 0.15" rpy="0 0 0"/>
+				<xacro:cylinder_inertia_def radius="0.03" length="0.30" mass="4.0" />
 		</inertial>
 		<visual>
-			<origin xyz="0 0 0.006" rpy="0 0 0"/>
+			<origin xyz="0 0 0.15" rpy="0 0 0"/>
 			<geometry>
-				<cylinder length="0.012" radius="0.035"/>
+				<cylinder length="0.30" radius="0.03"/>
 			</geometry>
 		</visual>
 		<collision>
-			<origin xyz="0 0 0.006" rpy="0 0 0"/>
+			<origin xyz="0 0 0.15" rpy="0 0 0"/>
 			<geometry>
-				<cylinder length="0.012" radius="0.035"/>
+				<cylinder length="0.30" radius="0.03"/>
 			</geometry>
 		</collision>
 	</link>
-	<gazebo reference="cylinder">
+	<gazebo reference="object_link">
+	    <material>Gazebo/Blue</material>
 		  <selfCollide>true</selfCollide>
 		 <maxContacts>100</maxContacts>
 	     <!-- <provideFeedback>true</provideFeedback>  -->
 	     <gravity>true</gravity>
-		<mu1>0.6</mu1>
+		<!-- <mu1>0.6</mu1>
+	     <mu2>0.6</mu2>
+	    -->
+	    <mu1>0.6</mu1>
 	     <mu2>0.6</mu2>
 	        <fdir1>1 0 0</fdir1>
          <maxVel>1.0</maxVel>
-		<kp>1000000000.0</kp>
-	  <kd>1000.0</kd>
+		<kp>1000000000000.0</kp>
+	  <kd>100000.0</kd>
 	  <minDepth>0.00</minDepth>
 	 </gazebo>
